File: Transmitter.kicad_sch (KiCad schematic)
At the start: 6 parts, among them U1 nRF24L01+, U2 Left Joystick, U3 Right Joystick, U4 AMS1117-3.3

Commit message: Update Transmitter.kicad_sch
Connections:
- net +5V: no longer U2.2 (VCC), U3.2 (VCC)
- net GND: no longer U2.4 (GND), U3.4 (GND)
- net PIN A0: no longer U2.3 (UP_DOWN)
- net PIN A1: no longer U2.1 (LEFT_RIGHT)
- net PIN A2: no longer U3.3 (UP_DOWN)
- net PIN A3: no longer U3.1 (LEFT_RIGHT)

Commit message: Update Transmitter.kicad_sch
Parts:
- removed U2: Left Joystick, symbol HackPackv4-cache:HackPackv4-rescue:PSP_1000_JSTK
- removed U3: Right Joystick, symbol HackPackv4-cache:HackPackv4-rescue:PSP_1000_JSTK
Changed lines of the file:
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@@
-	)
-	(symbol
-		(lib_id "HackPackv4-cache:HackPackv4-rescue:PSP_1000_JSTK")
-		(at 78.74 125.73 0)
-		(unit 1)
-		(exclude_from_sim no)
-		(in_bom yes)
-		(on_board yes)
-		(dnp no)
-		(fields_autoplaced yes)
-		(property "Reference" "U2"
-			(at 87.63 125.7299 0)
-			(effects
-				(font
-					(size 1.524 1.524)
-				)
-				(justify left)
-			)
-		)
-		(property "Value" "Left Joystick"
-			(at 87.63 128.2699 0)
-			(effects
-				(font
-					(size 1.524 1.524)
-				)
-				(justify left)
-			)
-		)
-		(property "Footprint" ""
-			(at 111.76 143.51 0)
-			(effects
-				(font
-					(size 1.524 1.524)
-				)
-				(hide yes)
-			)
-		)
-		(property "Datasheet" ""
-			(at 111.76 143.51 0)
-			(effects
-				(font
-					(size 1.524 1.524)
-				)
-				(hide yes)
-			)
-		)
-		(property "Description" ""
-			(at 78.74 125.73 0)
-			(effects
-				(font
-					(size 1.27 1.27)
-				)
-				(hide yes)
-			)
-		)
-		(pin "2"
-		)
-		(pin "3"
-		)
-		(pin "4"
-		)
-		(pin "1"
-		)
-		(instances
-			(project "Transmitter"
-				(path "/4266c96e-1acd-4150-949b-993f97093496"
-					(reference "U2")
-					(unit 1)
-				)
-			)
-		)
 	)
 	(symbol
@@
 					(unit 1)
 				)
-			)
-		)
-	)
-	(symbol
-		(lib_id "HackPackv4-cache:HackPackv4-rescue:PSP_1000_JSTK")
-		(at 205.74 125.73 0)
-		(unit 1)
-		(exclude_from_sim no)
-		(in_bom yes)
-		(on_board yes)
-		(dnp no)
-		(fields_autoplaced yes)
-		(property "Reference" "U3"
-			(at 214.63 125.7299 0)
-			(effects
-				(font
-					(size 1.524 1.524)
-				)
-				(justify left)
-			)
-		)
-		(property "Value" "Right Joystick"
-			(at 214.63 128.2699 0)
-			(effects
-				(font
-					(size 1.524 1.524)
-				)
-				(justify left)
-			)
-		)
-		(property "Footprint" ""
-			(at 238.76 143.51 0)
-			(effects
-				(font
-					(size 1.524 1.524)
-				)
-				(hide yes)
-			)
-		)
-		(property "Datasheet" ""
-			(at 238.76 143.51 0)
-			(effects
-				(font
-					(size 1.524 1.524)
-				)
-				(hide yes)
-			)
-		)
-		(property "Description" ""
-			(at 205.74 125.73 0)
-			(effects
-				(font
-					(size 1.27 1.27)
-				)
-				(hide yes)
-			)
-		)
-		(pin "3"
-		)
-		(pin "1"
-		)
-		(pin "4"
-		)
-		(pin "2"
-		)
-		(instances
-			(project "Transmitter"
-				(path "/4266c96e-1acd-4150-949b-993f97093496"
-					(reference "U3")
-					(unit 1)
-				)
